File: src/Issue 4.sch (KiCad schematic (older format))
At the start: 199 parts, among them IC1 ULA, IC10 4116, IC11 4116, IC12 4116, IC13 4116, IC14 LM1889, IC15 4532, IC16 4532, IC17 4532, IC18 4532, IC19 4532, IC2 Z80, IC20 4532, IC21 4532, IC22 4532, IC23 74LS32, IC24 74LS00, IC25 74LS157, IC26 74LS157, IC3 LS157, IC4 LS157, IC5 ROM, IC6 4116, IC7 4116, IC8 4116, IC9 4116, J1 OKI, J10 UR3, J11 UR4, J2 TI, J3 TI, J4 TI, J7 Barrel_Jack_MountingPin, J8 UR1, J9 UR2, T1 Coil, X1 14Mhz, X2 4.43Mhz

Commit message: 3d model of the coil
Parts:
- TV1: footprint Issue 4:Modulator -> (none)
Changed lines of the file:
@@
 	-1   0    0    1
 $EndComp
+Wire Wire Line
+	12100 5950 12100 8150
 $Comp
 L Issue-4-rescue:Modulator TV1
@@
 F 0 "TV1" H 3925 11665 50  0000 C CNN
 F 1 "Modulator" H 4100 11950 50  0000 C CNN
-F 2 "Issue 4:Modulator" H 4300 12050 50  0001 C CNN
+F 2 "" H 4300 12050 50  0001 C CNN
 F 3 "" H 4300 12050 50  0001 C CNN
 	1    4300 12050
@@
 Wire Wire Line
 	3550 11475 3550 11800
-Connection ~ 3250 11475
-Wire Wire Line
-	3250 11475 3250 11500
-Wire Wire Line
-	12100 5950 12100 8150
-Wire Wire Line
-	22550 8650 22550 9200
 Wire Wire Line
 	22650 8550 22650 9200
@@
 Wire Wire Line
 	23250 8650 23250 9200
-Wire Bus Line
-	20400 19800 24450 19800
 Wire Wire Line
 	11200 7250 11200 8150
@@
 Wire Bus Line
 	22350 8800 24450 8800
+Wire Wire Line
+	22550 8650 22550 9200
+Wire Bus Line
+	20400 19800 24450 19800
 Wire Bus Line
 	22250 18600 24450 18600
@@
 Wire Bus Line
 	10650 7750 12000 7750
+Connection ~ 3250 11475
+Wire Wire Line
+	3250 11475 3250 11500
 $EndSCHEMATC
